File: Backplane/Backplane.sch (KiCad schematic (older format))
At the start: 73 parts, among them U1 86093488314745V1LF, U10 86093488314745V1LF, U11 86093488314745V1LF, U12 86093488314745V1LF, U13 86093488314745V1LF, U14 86093488314745V1LF, U15 86093488314745V1LF, U16 86093488314745V1LF, U17 86093488314745V1LF, U18 86093488314745V1LF, U19 86093488314745V1LF, U2 86093488314745V1LF, U20 86093488314745V1LF, U21 74HC595, U22 74HC595, U23 74HC595, U24 74HC595, U25 74HC595, U26 74HC595, U27 74HC595, U28 74HC595, U29 74HC595, U3 86093488314745V1LF, U30 74HC595, U31 74HC595, U32 74HC595, U33 74HC595, U34 74HC595, U35 74HC595, U36 74HC595, U37 74HC595, U38 74HC595, U39 74HC595, U4 86093488314745V1LF, U40 74HC595, U5 86093488314745V1LF, U6 86093488314745V1LF, U7 86093488314745V1LF, U8 86093488314745V1LF, U9 86093488314745V1LF

Commit message: Rotate all connectors on the backplane (measure twice...)
Connections:
- net +3V3: now also U1.a15, U1.b15, U1.c15, U10.a15, U10.b15, U10.c15, U11.a15, U11.b15, U11.c15, U12.a15, U12.b15, U12.c15, U13.a15, U13.b15, U13.c15, U14.a15, U14.b15, U14.c15, U15.a15, U15.b15, U15.c15, U16.a15, U16.b15, U16.c15, U17.a15, U17.b15, U17.c15, U18.a15, U18.b15, U18.c15, U19.a15, U19.b15, U19.c15, U2.a15, U2.b15, U2.c15, U20.a15, U20.b15, U20.c15, U3.a15, U3.b15, U3.c15, U4.a15, U4.b15, U4.c15, U5.a15, U5.b15, U5.c15, U6.a15, U6.b15, U6.c15, U7.a15, U7.b15, U7.c15, U8.a15, U8.b15, U8.c15, U9.a15, U9.b15, U9.c15; no longer U1.a2, U1.b2, U1.c2, U10.a2, U10.b2, U10.c2, U11.a2, U11.b2, U11.c2, U12.a2, U12.b2, U12.c2, U13.a2, U13.b2, U13.c2, U14.a2, U14.b2, U14.c2, U15.a2, U15.b2, U15.c2, U16.a2, U16.b2, U16.c2, U17.a2, U17.b2, U17.c2, U18.a2, U18.b2, U18.c2, U19.a2, U19.b2, U19.c2, U2.a2, U2.b2, U2.c2, U20.a2, U20.b2, U20.c2, U3.a2, U3.b2, U3.c2, U4.a2, U4.b2, U4.c2, U5.a2, U5.b2, U5.c2, U6.a2, U6.b2, U6.c2, U7.a2, U7.b2, U7.c2, U8.a2, U8.b2, U8.c2, U9.a2, U9.b2, U9.c2
- net +5V: now also U1.a14, U1.b14, U1.c14, U10.a14, U10.b14, U10.c14, U11.a14, U11.b14, U11.c14, U12.a14, U12.b14, U12.c14, U13.a14, U13.b14, U13.c14, U14.a14, U14.b14, U14.c14, U15.a14, U15.b14, U15.c14, U16.a14, U16.b14, U16.c14, U17.a14, U17.b14, U17.c14, U18.a14, U18.b14, U18.c14, U19.a14, U19.b14, U19.c14, U2.a14, U2.b14, U2.c14, U20.a14, U20.b14, U20.c14, U3.a14, U3.b14, U3.c14, U4.a14, U4.b14, U4.c14, U5.a14, U5.b14, U5.c14, U6.a14, U6.b14, U6.c14, U7.a14, U7.b14, U7.c14, U8.a14, U8.b14, U8.c14, U9.a14, U9.b14, U9.c14; no longer U1.a3, U1.b3, U1.c3, U10.a3, U10.b3, U10.c3, U11.a3, U11.b3, U11.c3, U12.a3, U12.b3, U12.c3, U13.a3, U13.b3, U13.c3, U14.a3, U14.b3, U14.c3, U15.a3, U15.b3, U15.c3, U16.a3, U16.b3, U16.c3, U17.a3, U17.b3, U17.c3, U18.a3, U18.b3, U18.c3, U19.a3, U19.b3, U19.c3, U2.a3, U2.b3, U2.c3, U20.a3, U20.b3, U20.c3, U3.a3, U3.b3, U3.c3, U4.a3, U4.b3, U4.c3, U5.a3, U5.b3, U5.c3, U6.a3, U6.b3, U6.c3, U7.a3, U7.b3, U7.c3, U8.a3, U8.b3, U8.c3, U9.a3, U9.b3, U9.c3
- net DATA_IN_1: now also U18.c4, U20.a4; no longer U18.a13, U20.c13
- net EN_ICSP_1: now also U1.c3; no longer U1.a14
- net EN_ICSP_10: now also U5.a3; no longer U5.c14
- net EN_ICSP_11: now also U6.c3; no longer U6.a14
- net EN_ICSP_12: now also U6.a3; no longer U6.c14
- net EN_ICSP_13: now also U7.c3; no longer U7.a14
- net EN_ICSP_14: now also U7.a3; no longer U7.c14
- net EN_ICSP_15: now also U8.c3; no longer U8.a14
- net EN_ICSP_16: now also U8.a3; no longer U8.c14
- net EN_ICSP_17: now also U9.c3; no longer U9.a14
- net EN_ICSP_18: now also U9.a3; no longer U9.c14
- net EN_ICSP_19: now also U10.c3; no longer U10.a14
- net EN_ICSP_2: now also U1.a3; no longer U1.c14
- net EN_ICSP_20: now also U10.a3; no longer U10.c14
- net EN_ICSP_21: now also U11.c3; no longer U11.a14
- net EN_ICSP_22: now also U11.a3; no longer U11.c14
- net EN_ICSP_23: now also U12.c3; no longer U12.a14
- net EN_ICSP_24: now also U12.a3; no longer U12.c14
- net EN_ICSP_25: now also U13.c3; no longer U13.a14
- net EN_ICSP_26: now also U13.a3; no longer U13.c14
- net EN_ICSP_27: now also U14.c3; no longer U14.a14
- net EN_ICSP_28: now also U14.a3; no longer U14.c14
- net EN_ICSP_29: now also U15.c3; no longer U15.a14
- net EN_ICSP_3: now also U2.c3; no longer U2.a14
- net EN_ICSP_30: now also U15.a3; no longer U15.c14
- net EN_ICSP_31: now also U16.c3; no longer U16.a14
- net EN_ICSP_32: now also U16.a3; no longer U16.c14
- net EN_ICSP_33: now also U17.c3; no longer U17.a14
- net EN_ICSP_34: now also U17.a3; no longer U17.c14
- net EN_ICSP_36: now also U18.a3; no longer U18.c14
- net EN_ICSP_37: now also U19.c3; no longer U19.a14
- net EN_ICSP_39: now also U20.c3; no longer U20.a14
- net EN_ICSP_4: now also U2.a3; no longer U2.c14
- net EN_ICSP_5: now also U3.c3; no longer U3.a14
- net EN_ICSP_6: now also U3.a3; no longer U3.c14
- net EN_ICSP_7: now also U4.c3; no longer U4.a14
- net EN_ICSP_8: now also U4.a3; no longer U4.c14
- net EN_ICSP_9: now also U5.c3; no longer U5.a14
- net EN_JTAG_1: now also U1.c2; no longer U1.a15
- net EN_JTAG_10: now also U5.a2; no longer U5.c15
- net EN_JTAG_11: now also U6.c2; no longer U6.a15
- net EN_JTAG_12: now also U6.a2; no longer U6.c15
- net EN_JTAG_13: now also U7.c2; no longer U7.a15
- net EN_JTAG_14: now also U7.a2; no longer U7.c15
- net EN_JTAG_15: now also U8.c2; no longer U8.a15
- net EN_JTAG_16: now also U8.a2; no longer U8.c15
- net EN_JTAG_17: now also U9.c2; no longer U9.a15
- net EN_JTAG_18: now also U9.a2; no longer U9.c15
- net EN_JTAG_19: now also U10.c2; no longer U10.a15
- net EN_JTAG_2: now also U1.a2; no longer U1.c15
- net EN_JTAG_20: now also U10.a2; no longer U10.c15
- net EN_JTAG_21: now also U11.c2; no longer U11.a15
- net EN_JTAG_22: now also U11.a2; no longer U11.c15
- net EN_JTAG_23: now also U12.c2; no longer U12.a15
- net EN_JTAG_24: now also U12.a2; no longer U12.c15
- net EN_JTAG_25: now also U13.c2; no longer U13.a15
- net EN_JTAG_26: now also U13.a2; no longer U13.c15
- net EN_JTAG_27: now also U14.c2; no longer U14.a15
- net EN_JTAG_28: now also U14.a2; no longer U14.c15
- net EN_JTAG_29: now also U15.c2; no longer U15.a15
- net EN_JTAG_3: now also U2.c2; no longer U2.a15
- net EN_JTAG_30: now also U15.a2; no longer U15.c15
- net EN_JTAG_31: now also U16.c2; no longer U16.a15
- net EN_JTAG_32: now also U16.a2; no longer U16.c15
- net EN_JTAG_33: now also U17.c2; no longer U17.a15
- net EN_JTAG_34: now also U17.a2; no longer U17.c15
- net EN_JTAG_36: now also U18.a2; no longer U18.c15
- net EN_JTAG_37: now also U19.c2; no longer U19.a15
- net EN_JTAG_39: now also U20.c2; no longer U20.a15
- net EN_JTAG_4: now also U2.a2; no longer U2.c15
- net EN_JTAG_5: now also U3.c2; no longer U3.a15
- net EN_JTAG_6: now also U3.a2; no longer U3.c15
- net EN_JTAG_7: now also U4.c2; no longer U4.a15
- net EN_JTAG_8: now also U4.a2; no longer U4.c15
- net EN_JTAG_9: now also U5.c2; no longer U5.a15
- net EN_PWR_1: now also U1.c4; no longer U1.a13
- net EN_PWR_10: now also U5.a4; no longer U5.c13
- net EN_PWR_11: now also U6.c4; no longer U6.a13
- net EN_PWR_12: now also U6.a4; no longer U6.c13
- net EN_PWR_13: now also U7.c4; no longer U7.a13
- net EN_PWR_14: now also U7.a4; no longer U7.c13
- net EN_PWR_15: now also U8.c4; no longer U8.a13
- net EN_PWR_16: now also U8.a4; no longer U8.c13
- net EN_PWR_17: now also U9.c4; no longer U9.a13
- net EN_PWR_18: now also U9.a4; no longer U9.c13
- net EN_PWR_19: now also U10.c4; no longer U10.a13
- net EN_PWR_2: now also U1.a4; no longer U1.c13
- net EN_PWR_20: now also U10.a4; no longer U10.c13
- net EN_PWR_21: now also U11.c4; no longer U11.a13
- net EN_PWR_22: now also U11.a4; no longer U11.c13
- net EN_PWR_23: now also U12.c4; no longer U12.a13
- net EN_PWR_24: now also U12.a4; no longer U12.c13
- net EN_PWR_25: now also U13.c4; no longer U13.a13
- net EN_PWR_26: now also U13.a4; no longer U13.c13
- net EN_PWR_27: now also U14.c4; no longer U14.a13
- net EN_PWR_28: now also U14.a4; no longer U14.c13
- net EN_PWR_29: now also U15.c4; no longer U15.a13
- net EN_PWR_3: now also U2.c4; no longer U2.a13
- net EN_PWR_30: now also U15.a4; no longer U15.c13
- net EN_PWR_31: now also U16.c4; no longer U16.a13
- net EN_PWR_32: now also U16.a4; no longer U16.c13
- net EN_PWR_33: now also U17.c4; no longer U17.a13
- net EN_PWR_34: now also U17.a4; no longer U17.c13
- net EN_PWR_37: now also U19.c4; no longer U19.a13
- net EN_PWR_39: now also U20.c4; no longer U20.a13
- net EN_PWR_4: now also U2.a4; no longer U2.c13
- net EN_PWR_5: now also U3.c4; no longer U3.a13
- net EN_PWR_6: now also U3.a4; no longer U3.c13
- net EN_PWR_7: now also U4.c4; no longer U4.a13
- net EN_PWR_8: now also U4.a4; no longer U4.c13
- net EN_PWR_9: now also U5.c4; no longer U5.a13
- net GND: now also U1.a16, U1.b16, U1.c16, U10.a16, U10.b16, U10.c16, U11.a16, U11.b16, U11.c16, U12.a16, U12.b16, U12.c16, U13.a16, U13.b16, U13.c16, U14.a16, U14.b16, U14.c16, U15.a16, U15.b16, U15.c16, U16.a16, U16.b16, U16.c16, U17.a16, U17.b16, U17.c16, U18.a16, U18.b16, U18.c16, U19.a16, U19.b16, U19.c16, U2.a16, U2.b16, U2.c16, U20.a16, U20.b16, U20.c16, U3.a16, U3.b16, U3.c16, U4.a16, U4.b16, U4.c16, U5.a16, U5.b16, U5.c16, U6.a16, U6.b16, U6.c16, U7.a16, U7.b16, U7.c16, U8.a16, U8.b16, U8.c16, U9.a16, U9.b16, U9.c16; no longer U1.a1, U1.b1, U1.c1, U10.a1, U10.b1, U10.c1, U11.a1, U11.b1, U11.c1, U12.a1, U12.b1, U12.c1, U13.a1, U13.b1, U13.c1, U14.a1, U14.b1, U14.c1, U15.a1, U15.b1, U15.c1, U16.a1, U16.b1, U16.c1, U17.a1, U17.b1, U17.c1, U18.a1, U18.b1, U18.c1, U19.a1, U19.b1, U19.c1, U2.a1, U2.b1, U2.c1, U20.a1, U20.b1, U20.c1, U3.a1, U3.b1, U3.c1, U4.a1, U4.b1, U4.c1, U5.a1, U5.b1, U5.c1, U6.a1, U6.b1, U6.c1, U7.a1, U7.b1, U7.c1, U8.a1, U8.b1, U8.c1, U9.a1, U9.b1, U9.c1
- net PGEC: now also U1.a8, U1.b8, U1.c8, U10.a8, U10.b8, U10.c8, U11.a8, U11.b8, U11.c8, U12.a8, U12.b8, U12.c8, U13.a8, U13.b8, U13.c8, U14.a8, U14.b8, U14.c8, U15.a8, U15.b8, U15.c8, U16.a8, U16.b8, U16.c8, U17.a8, U17.b8, U17.c8, U18.a8, U18.b8, U18.c8, U19.c8, U2.a8, U2.b8, U2.c8, U20.c8, U3.a8, U3.b8, U3.c8, U4.a8, U4.b8, U4.c8, U5.a8, U5.b8, U5.c8, U6.a8, U6.b8, U6.c8, U7.a8, U7.b8, U7.c8, U8.a8, U8.b8, U8.c8, U9.a8, U9.b8, U9.c8; no longer U1.a9, U1.b9, U1.c9, U10.a9, U10.b9, U10.c9, U11.a9, U11.b9, U11.c9, U12.a9, U12.b9, U12.c9, U13.a9, U13.b9, U13.c9, U14.a9, U14.b9, U14.c9, U15.a9, U15.b9, U15.c9, U16.a9, U16.b9, U16.c9, U17.a9, U17.b9, U17.c9, U18.a9, U18.b9, U18.c9, U19.a9, U2.a9, U2.b9, U2.c9, U20.a9, U3.a9, U3.b9, U3.c9, U4.a9, U4.b9, U4.c9, U5.a9, U5.b9, U5.c9, U6.a9, U6.b9, U6.c9, U7.a9, U7.b9, U7.c9, U8.a9, U8.b9, U8.c9, U9.a9, U9.b9, U9.c9
- net PGED: now also U1.a7, U1.b7, U1.c7, U10.a7, U10.b7, U10.c7, U11.a7, U11.b7, U11.c7, U12.a7, U12.b7, U12.c7, U13.a7, U13.b7, U13.c7, U14.a7, U14.b7, U14.c7, U15.a7, U15.b7, U15.c7, U16.a7, U16.b7, U16.c7, U17.a7, U17.b7, U17.c7, U18.a7, U18.b7, U18.c7, U19.c7, U2.a7, U2.b7, U2.c7, U20.c7, U3.a7, U3.b7, U3.c7, U4.a7, U4.b7, U4.c7, U5.a7, U5.b7, U5.c7, U6.a7, U6.b7, U6.c7, U7.a7, U7.b7, U7.c7, U8.a7, U8.b7, U8.c7, U9.a7, U9.b7, U9.c7; no longer U1.a10, U1.b10, U1.c10, U10.a10, U10.b10, U10.c10, U11.a10, U11.b10, U11.c10, U12.a10, U12.b10, U12.c10, U13.a10, U13.b10, U13.c10, U14.a10, U14.b10, U14.c10, U15.a10, U15.b10, U15.c10, U16.a10, U16.b10, U16.c10, U17.a10, U17.b10, U17.c10, U18.a10, U18.b10, U18.c10, U19.a10, U2.a10, U2.b10, U2.c10, U20.a10, U3.a10, U3.b10, U3.c10, U4.a10, U4.b10, U4.c10, U5.a10, U5.b10, U5.c10, U6.a10, U6.b10, U6.c10, U7.a10, U7.b10, U7.c10, U8.a10, U8.b10, U8.c10, U9.a10, U9.b10, U9.c10
- net SHIFT_CLK_IN: now also U18.c3, U20.a3; no longer U18.a14, U20.c14
- net SPARE_1: now also U1.c1; no longer U1.a16
- net SPARE_10: now also U5.a1; no longer U5.c16
- net SPARE_11: now also U6.c1; no longer U6.a16
- net SPARE_12: now also U6.a1; no longer U6.c16
- net SPARE_13: now also U7.c1; no longer U7.a16
- net SPARE_14: now also U7.a1; no longer U7.c16
- net SPARE_15: now also U8.c1; no longer U8.a16
- net SPARE_16: now also U8.a1; no longer U8.c16
- net SPARE_17: now also U9.c1; no longer U9.a16
- net SPARE_18: now also U9.a1; no longer U9.c16
- net SPARE_19: now also U10.c1; no longer U10.a16
- net SPARE_2: now also U1.a1; no longer U1.c16
- net SPARE_20: now also U10.a1; no longer U10.c16
- net SPARE_21: now also U11.c1; no longer U11.a16
- net SPARE_22: now also U11.a1; no longer U11.c16
- net SPARE_23: now also U12.c1; no longer U12.a16
- net SPARE_24: now also U12.a1; no longer U12.c16
- net SPARE_25: now also U13.c1; no longer U13.a16
- net SPARE_26: now also U13.a1; no longer U13.c16
- net SPARE_27: now also U14.c1; no longer U14.a16
- net SPARE_28: now also U14.a1; no longer U14.c16
- net SPARE_29: now also U15.c1; no longer U15.a16
- net SPARE_3: now also U2.c1; no longer U2.a16
- net SPARE_30: now also U15.a1; no longer U15.c16
- net SPARE_31: now also U16.c1; no longer U16.a16
- net SPARE_32: now also U16.a1; no longer U16.c16
- net SPARE_33: now also U17.c1; no longer U17.a16
- net SPARE_34: now also U17.a1; no longer U17.c16
- net SPARE_37: now also U19.c1; no longer U19.a16
- net SPARE_39: now also U20.c1; no longer U20.a16
- net SPARE_4: now also U2.a1; no longer U2.c16
- net SPARE_5: now also U3.c1; no longer U3.a16
- net SPARE_6: now also U3.a1; no longer U3.c16
- net SPARE_7: now also U4.c1; no longer U4.a16
- net SPARE_8: now also U4.a1; no longer U4.c16
- net SPARE_9: now also U5.c1; no longer U5.a16
- net STORAGE_CLK: now also U18.c2, U20.a2; no longer U18.a15, U20.c15
- net TARGET_RX: now also U1.a6, U1.b6, U1.c6, U10.a6, U10.b6, U10.c6, U11.a6, U11.b6, U11.c6, U12.a6, U12.b6, U12.c6, U13.a6, U13.b6, U13.c6, U14.a6, U14.b6, U14.c6, U15.a6, U15.b6, U15.c6, U16.a6, U16.b6, U16.c6, U17.a6, U17.b6, U17.c6, U18.a6, U18.b6, U18.c6, U19.c6, U2.a6, U2.b6, U2.c6, U20.c6, U3.a6, U3.b6, U3.c6, U4.a6, U4.b6, U4.c6, U5.a6, U5.b6, U5.c6, U6.a6, U6.b6, U6.c6, U7.a6, U7.b6, U7.c6, U8.a6, U8.b6, U8.c6, U9.a6, U9.b6, U9.c6; no longer U1.a11, U1.b11, U1.c11, U10.a11, U10.b11, U10.c11, U11.a11, U11.b11, U11.c11, U12.a11, U12.b11, U12.c11, U13.a11, U13.b11, U13.c11, U14.a11, U14.b11, U14.c11, U15.a11, U15.b11, U15.c11, U16.a11, U16.b11, U16.c11, U17.a11, U17.b11, U17.c11, U18.a11, U18.b11, U18.c11, U19.a11, U2.a11, U2.b11, U2.c11, U20.a11, U3.a11, U3.b11, U3.c11, U4.a11, U4.b11, U4.c11, U5.a11, U5.b11, U5.c11, U6.a11, U6.b11, U6.c11, U7.a11, U7.b11, U7.c11, U8.a11, U8.b11, U8.c11, U9.a11, U9.b11, U9.c11
- net TARGET_TX: now also U1.a5, U1.b5, U1.c5, U10.a5, U10.b5, U10.c5, U11.a5, U11.b5, U11.c5, U12.a5, U12.b5, U12.c5, U13.a5, U13.b5, U13.c5, U14.a5, U14.b5, U14.c5, U15.a5, U15.b5, U15.c5, U16.a5, U16.b5, U16.c5, U17.a5, U17.b5, U17.c5, U18.a5, U18.b5, U18.c5, U19.c5, U2.a5, U2.b5, U2.c5, U20.c5, U3.a5, U3.b5, U3.c5, U4.a5, U4.b5, U4.c5, U5.a5, U5.b5, U5.c5, U6.a5, U6.b5, U6.c5, U7.a5, U7.b5, U7.c5, U8.a5, U8.b5, U8.c5, U9.a5, U9.b5, U9.c5; no longer U1.a12, U1.b12, U1.c12, U10.a12, U10.b12, U10.c12, U11.a12, U11.b12, U11.c12, U12.a12, U12.b12, U12.c12, U13.a12, U13.b12, U13.c12, U14.a12, U14.b12, U14.c12, U15.a12, U15.b12, U15.c12, U16.a12, U16.b12, U16.c12, U17.a12, U17.b12, U17.c12, U18.a12, U18.b12, U18.c12, U19.a12, U2.a12, U2.b12, U2.c12, U20.a12, U3.a12, U3.b12, U3.c12, U4.a12, U4.b12, U4.c12, U5.a12, U5.b12, U5.c12, U6.a12, U6.b12, U6.c12, U7.a12, U7.b12, U7.c12, U8.a12, U8.b12, U8.c12, U9.a12, U9.b12, U9.c12
- net TCK: now also U1.a10, U1.b10, U1.c10, U10.a10, U10.b10, U10.c10, U11.a10, U11.b10, U11.c10, U12.a10, U12.b10, U12.c10, U13.a10, U13.b10, U13.c10, U14.a10, U14.b10, U14.c10, U15.a10, U15.b10, U15.c10, U16.a10, U16.b10, U16.c10, U17.a10, U17.b10, U17.c10, U18.a10, U18.b10, U18.c10, U19.c10, U2.a10, U2.b10, U2.c10, U20.c10, U3.a10, U3.b10, U3.c10, U4.a10, U4.b10, U4.c10, U5.a10, U5.b10, U5.c10, U6.a10, U6.b10, U6.c10, U7.a10, U7.b10, U7.c10, U8.a10, U8.b10, U8.c10, U9.a10, U9.b10, U9.c10; no longer U1.a7, U1.b7, U1.c7, U10.a7, U10.b7, U10.c7, U11.a7, U11.b7, U11.c7, U12.a7, U12.b7, U12.c7, U13.a7, U13.b7, U13.c7, U14.a7, U14.b7, U14.c7, U15.a7, U15.b7, U15.c7, U16.a7, U16.b7, U16.c7, U17.a7, U17.b7, U17.c7, U18.a7, U18.b7, U18.c7, U19.a7, U2.a7, U2.b7, U2.c7, U20.a7, U3.a7, U3.b7, U3.c7, U4.a7, U4.b7, U4.c7, U5.a7, U5.b7, U5.c7, U6.a7, U6.b7, U6.c7, U7.a7, U7.b7, U7.c7, U8.a7, U8.b7, U8.c7, U9.a7, U9.b7, U9.c7
- net TDI: now also U1.a13, U1.b13, U1.c13, U10.a13, U10.b13, U10.c13, U11.a13, U11.b13, U11.c13, U12.a13, U12.b13, U12.c13, U13.a13, U13.b13, U13.c13, U14.a13, U14.b13, U14.c13, U15.a13, U15.b13, U15.c13, U16.a13, U16.b13, U16.c13, U17.a13, U17.b13, U17.c13, U18.a13, U18.b13, U18.c13, U19.c13, U2.a13, U2.b13, U2.c13, U20.c13, U3.a13, U3.b13, U3.c13, U4.a13, U4.b13, U4.c13, U5.a13, U5.b13, U5.c13, U6.a13, U6.b13, U6.c13, U7.a13, U7.b13, U7.c13, U8.a13, U8.b13, U8.c13, U9.a13, U9.b13, U9.c13; no longer U1.a4, U1.b4, U1.c4, U10.a4, U10.b4, U10.c4, U11.a4, U11.b4, U11.c4, U12.a4, U12.b4, U12.c4, U13.a4, U13.b4, U13.c4, U14.a4, U14.b4, U14.c4, U15.a4, U15.b4, U15.c4, U16.a4, U16.b4, U16.c4, U17.a4, U17.b4, U17.c4, U18.a4, U18.b4, U18.c4, U19.a4, U2.a4, U2.b4, U2.c4, U20.a4, U3.a4, U3.b4, U3.c4, U4.a4, U4.b4, U4.c4, U5.a4, U5.b4, U5.c4, U6.a4, U6.b4, U6.c4, U7.a4, U7.b4, U7.c4, U8.a4, U8.b4, U8.c4, U9.a4, U9.b4, U9.c4
- net TDO: now also U1.a12, U1.b12, U1.c12, U10.a12, U10.b12, U10.c12, U11.a12, U11.b12, U11.c12, U12.a12, U12.b12, U12.c12, U13.a12, U13.b12, U13.c12, U14.a12, U14.b12, U14.c12, U15.a12, U15.b12, U15.c12, U16.a12, U16.b12, U16.c12, U17.a12, U17.b12, U17.c12, U18.a12, U18.b12, U18.c12, U19.c12, U2.a12, U2.b12, U2.c12, U20.c12, U3.a12, U3.b12, U3.c12, U4.a12, U4.b12, U4.c12, U5.a12, U5.b12, U5.c12, U6.a12, U6.b12, U6.c12, U7.a12, U7.b12, U7.c12, U8.a12, U8.b12, U8.c12, U9.a12, U9.b12, U9.c12; no longer U1.a5, U1.b5, U1.c5, U10.a5, U10.b5, U10.c5, U11.a5, U11.b5, U11.c5, U12.a5, U12.b5, U12.c5, U13.a5, U13.b5, U13.c5, U14.a5, U14.b5, U14.c5, U15.a5, U15.b5, U15.c5, U16.a5, U16.b5, U16.c5, U17.a5, U17.b5, U17.c5, U18.a5, U18.b5, U18.c5, U19.a5, U2.a5, U2.b5, U2.c5, U20.a5, U3.a5, U3.b5, U3.c5, U4.a5, U4.b5, U4.c5, U5.a5, U5.b5, U5.c5, U6.a5, U6.b5, U6.c5, U7.a5, U7.b5, U7.c5, U8.a5, U8.b5, U8.c5, U9.a5, U9.b5, U9.c5
- net TMS: now also U1.a11, U1.b11, U1.c11, U10.a11, U10.b11, U10.c11, U11.a11, U11.b11, U11.c11, U12.a11, U12.b11, U12.c11, U13.a11, U13.b11, U13.c11, U14.a11, U14.b11, U14.c11, U15.a11, U15.b11, U15.c11, U16.a11, U16.b11, U16.c11, U17.a11, U17.b11, U17.c11, U18.a11, U18.b11, U18.c11, U19.c11, U2.a11, U2.b11, U2.c11, U20.c11, U3.a11, U3.b11, U3.c11, U4.a11, U4.b11, U4.c11, U5.a11, U5.b11, U5.c11, U6.a11, U6.b11, U6.c11, U7.a11, U7.b11, U7.c11, U8.a11, U8.b11, U8.c11, U9.a11, U9.b11, U9.c11; no longer U1.a6, U1.b6, U1.c6, U10.a6, U10.b6, U10.c6, U11.a6, U11.b6, U11.c6, U12.a6, U12.b6, U12.c6, U13.a6, U13.b6, U13.c6, U14.a6, U14.b6, U14.c6, U15.a6, U15.b6, U15.c6, U16.a6, U16.b6, U16.c6, U17.a6, U17.b6, U17.c6, U18.a6, U18.b6, U18.c6, U19.a6, U2.a6, U2.b6, U2.c6, U20.a6, U3.a6, U3.b6, U3.c6, U4.a6, U4.b6, U4.c6, U5.a6, U5.b6, U5.c6, U6.a6, U6.b6, U6.c6, U7.a6, U7.b6, U7.c6, U8.a6, U8.b6, U8.c6, U9.a6, U9.b6, U9.c6
- net ~MASTER_RST~: now also U18.a4, U20.a5; no longer U18.c13, U20.c12
- net ~MCLR~: now also U1.a9, U1.b9, U1.c9, U10.a9, U10.b9, U10.c9, U11.a9, U11.b9, U11.c9, U12.a9, U12.b9, U12.c9, U13.a9, U13.b9, U13.c9, U14.a9, U14.b9, U14.c9, U15.a9, U15.b9, U15.c9, U16.a9, U16.b9, U16.c9, U17.a9, U17.b9, U17.c9, U18.a9, U18.b9, U18.c9, U19.c9, U2.a9, U2.b9, U2.c9, U20.c9, U3.a9, U3.b9, U3.c9, U4.a9, U4.b9, U4.c9, U5.a9, U5.b9, U5.c9, U6.a9, U6.b9, U6.c9, U7.a9, U7.b9, U7.c9, U8.a9, U8.b9, U8.c9, U9.a9, U9.b9, U9.c9; no longer U1.a8, U1.b8, U1.c8, U10.a8, U10.b8, U10.c8, U11.a8, U11.b8, U11.c8, U12.a8, U12.b8, U12.c8, U13.a8, U13.b8, U13.c8, U14.a8, U14.b8, U14.c8, U15.a8, U15.b8, U15.c8, U16.a8, U16.b8, U16.c8, U17.a8, U17.b8, U17.c8, U18.a8, U18.b8, U18.c8, U19.a8, U2.a8, U2.b8, U2.c8, U20.a8, U3.a8, U3.b8, U3.c8, U4.a8, U4.b8, U4.c8, U5.a8, U5.b8, U5.c8, U6.a8, U6.b8, U6.c8, U7.a8, U7.b8, U7.c8, U8.a8, U8.b8, U8.c8, U9.a8, U9.b8, U9.c8
- net ~OE~: now also U18.c1, U20.a1; no longer U18.a16, U20.c16
