File: Backplane/Backplane.kicad_pcb (KiCad board)
At the start: 2 copper layers, 412 x 76 mm, 73 parts, among them U1 86093488314745V1LF, U10 86093488314745V1LF, U11 86093488314745V1LF, U12 86093488314745V1LF, U13 86093488314745V1LF, U14 86093488314745V1LF, U15 86093488314745V1LF, U16 86093488314745V1LF, U17 86093488314745V1LF, U18 86093488314745V1LF, U19 86093488314745V1LF, U2 86093488314745V1LF, U20 86093488314745V1LF, U21 74HC595, U22 74HC595, U23 74HC595, U24 74HC595, U25 74HC595, U26 74HC595, U27 74HC595, U28 74HC595, U29 74HC595, U3 86093488314745V1LF, U30 74HC595, U31 74HC595, U32 74HC595, U33 74HC595, U34 74HC595, U35 74HC595, U36 74HC595, U37 74HC595, U38 74HC595, U39 74HC595, U4 86093488314745V1LF, U40 74HC595, U5 86093488314745V1LF, U6 86093488314745V1LF, U7 86093488314745V1LF, U8 86093488314745V1LF, U9 86093488314745V1LF

Commit message: Rotate all connectors on the backplane (measure twice...)
Parts:
- moved U15 38.4 mm to (344.5, 107.1), turned to 180 degrees
- moved U2 38.4 mm to (76.7, 107.1), turned to 180 degrees
- moved U20 38.4 mm to (447.5, 107.1), turned to 180 degrees
- moved U6 38.4 mm to (159.1, 107.1), turned to 180 degrees
- moved U7 38.4 mm to (179.7, 107.1), turned to 180 degrees
- moved U8 38.4 mm to (200.3, 107.1), turned to 180 degrees
- moved U1 38.4 mm to (56.1, 107.1), turned to 180 degrees
- moved U10 38.4 mm to (241.5, 107.1), turned to 180 degrees
- moved U11 38.4 mm to (262.1, 107.1), turned to 180 degrees
- moved U12 38.4 mm to (282.7, 107.1), turned to 180 degrees
- moved U13 38.4 mm to (303.3, 107.1), turned to 180 degrees
- moved U14 38.4 mm to (323.9, 107.1), turned to 180 degrees
- moved U16 38.4 mm to (365.1, 107.1), turned to 180 degrees
- moved U17 38.4 mm to (385.7, 107.1), turned to 180 degrees
- moved U18 38.4 mm to (406.3, 107.1), turned to 180 degrees
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Connections:
- U1 pad a1: GND -> /SPARE_2
- U1 pad a10: /PGED -> /TCK
- U1 pad a11: /TARGET_RX -> /TMS
- U1 pad a12: /TARGET_TX -> /TDO
- U1 pad a13: /EN_PWR_1 -> /TDI
- U1 pad a14: /EN_ICSP_1 -> +5V
- U1 pad a15: /EN_JTAG_1 -> +3V3
- U1 pad a16: /SPARE_1 -> GND
- U1 pad a2: +3V3 -> /EN_JTAG_2
- U1 pad a3: +5V -> /EN_ICSP_2
- U1 pad a4: /TDI -> /EN_PWR_2
- U1 pad a5: /TDO -> /TARGET_TX
- U1 pad a6: /TMS -> /TARGET_RX
- U1 pad a7: /TCK -> /PGED
- U1 pad a8: /~MCLR~ -> /PGEC
- U1 pad a9: /PGEC -> /~MCLR~
- U1 pad b1: GND -> (no net)
- U1 pad b10: /PGED -> /TCK
- U1 pad b11: /TARGET_RX -> /TMS
- U1 pad b12: /TARGET_TX -> /TDO
- U1 pad b13: (no net) -> /TDI
- U1 pad b14: (no net) -> +5V
- U1 pad b15: (no net) -> +3V3
- U1 pad b16: (no net) -> GND
- U1 pad b2: +3V3 -> (no net)
- U1 pad b3: +5V -> (no net)
- U1 pad b4: /TDI -> (no net)
- U1 pad b5: /TDO -> /TARGET_TX
- U1 pad b6: /TMS -> /TARGET_RX
- U1 pad b7: /TCK -> /PGED
- U1 pad b8: /~MCLR~ -> /PGEC
- U1 pad b9: /PGEC -> /~MCLR~
- U1 pad c1: GND -> /SPARE_1
- U1 pad c10: /PGED -> /TCK
- U1 pad c11: /TARGET_RX -> /TMS
- U1 pad c12: /TARGET_TX -> /TDO
- U1 pad c13: /EN_PWR_2 -> /TDI
- U1 pad c14: /EN_ICSP_2 -> +5V
- U1 pad c15: /EN_JTAG_2 -> +3V3
- U1 pad c16: /SPARE_2 -> GND
- U1 pad c2: +3V3 -> /EN_JTAG_1
- U1 pad c3: +5V -> /EN_ICSP_1
- U1 pad c4: /TDI -> /EN_PWR_1
- U1 pad c5: /TDO -> /TARGET_TX
- U1 pad c6: /TMS -> /TARGET_RX
- U1 pad c7: /TCK -> /PGED
- U1 pad c8: /~MCLR~ -> /PGEC
- U1 pad c9: /PGEC -> /~MCLR~
- U10 pad a1: GND -> /SPARE_20
- U10 pad a10: /PGED -> /TCK
- U10 pad a11: /TARGET_RX -> /TMS
- U10 pad a12: /TARGET_TX -> /TDO
- U10 pad a13: /EN_PWR_19 -> /TDI
- U10 pad a14: /EN_ICSP_19 -> +5V
- U10 pad a15: /EN_JTAG_19 -> +3V3
- U10 pad a16: /SPARE_19 -> GND
- U10 pad a2: +3V3 -> /EN_JTAG_20
- U10 pad a3: +5V -> /EN_ICSP_20
- U10 pad a4: /TDI -> /EN_PWR_20
- U10 pad a5: /TDO -> /TARGET_TX
- U10 pad a6: /TMS -> /TARGET_RX
- U10 pad a7: /TCK -> /PGED
- U10 pad a8: /~MCLR~ -> /PGEC
- U10 pad a9: /PGEC -> /~MCLR~
- U10 pad b1: GND -> (no net)
- U10 pad b10: /PGED -> /TCK
- U10 pad b11: /TARGET_RX -> /TMS
- U10 pad b12: /TARGET_TX -> /TDO
- U10 pad b13: (no net) -> /TDI
- U10 pad b14: (no net) -> +5V
- U10 pad b15: (no net) -> +3V3
- U10 pad b16: (no net) -> GND
- U10 pad b2: +3V3 -> (no net)
- U10 pad b3: +5V -> (no net)
- U10 pad b4: /TDI -> (no net)
- U10 pad b5: /TDO -> /TARGET_TX
- U10 pad b6: /TMS -> /TARGET_RX
- U10 pad b7: /TCK -> /PGED
- U10 pad b8: /~MCLR~ -> /PGEC
- U10 pad b9: /PGEC -> /~MCLR~
- U10 pad c1: GND -> /SPARE_19
- U10 pad c10: /PGED -> /TCK
- U10 pad c11: /TARGET_RX -> /TMS
- U10 pad c12: /TARGET_TX -> /TDO
- U10 pad c13: /EN_PWR_20 -> /TDI
- U10 pad c14: /EN_ICSP_20 -> +5V
- U10 pad c15: /EN_JTAG_20 -> +3V3
- U10 pad c16: /SPARE_20 -> GND
- U10 pad c2: +3V3 -> /EN_JTAG_19
- U10 pad c3: +5V -> /EN_ICSP_19
- U10 pad c4: /TDI -> /EN_PWR_19
- U10 pad c5: /TDO -> /TARGET_TX
- U10 pad c6: /TMS -> /TARGET_RX
- U10 pad c7: /TCK -> /PGED
- U10 pad c8: /~MCLR~ -> /PGEC
- U10 pad c9: /PGEC -> /~MCLR~
- U11 pad a1: GND -> /SPARE_22
- U11 pad a10: /PGED -> /TCK
- U11 pad a11: /TARGET_RX -> /TMS
- U11 pad a12: /TARGET_TX -> /TDO
- U11 pad a13: /EN_PWR_21 -> /TDI
- U11 pad a14: /EN_ICSP_21 -> +5V
- U11 pad a15: /EN_JTAG_21 -> +3V3
- U11 pad a16: /SPARE_21 -> GND
- U11 pad a2: +3V3 -> /EN_JTAG_22
- U11 pad a3: +5V -> /EN_ICSP_22
- U11 pad a4: /TDI -> /EN_PWR_22
- U11 pad a5: /TDO -> /TARGET_TX
- U11 pad a6: /TMS -> /TARGET_RX
- U11 pad a7: /TCK -> /PGED
- U11 pad a8: /~MCLR~ -> /PGEC
- U11 pad a9: /PGEC -> /~MCLR~
- U11 pad b1: GND -> (no net)
- U11 pad b10: /PGED -> /TCK
- U11 pad b11: /TARGET_RX -> /TMS
- U11 pad b12: /TARGET_TX -> /TDO
- U11 pad b13: (no net) -> /TDI
- U11 pad b14: (no net) -> +5V
- U11 pad b15: (no net) -> +3V3
- U11 pad b16: (no net) -> GND
- U11 pad b2: +3V3 -> (no net)
- U11 pad b3: +5V -> (no net)
- U11 pad b4: /TDI -> (no net)
- U11 pad b5: /TDO -> /TARGET_TX
- U11 pad b6: /TMS -> /TARGET_RX
- U11 pad b7: /TCK -> /PGED
- U11 pad b8: /~MCLR~ -> /PGEC
- U11 pad b9: /PGEC -> /~MCLR~
- U11 pad c1: GND -> /SPARE_21
- U11 pad c10: /PGED -> /TCK
- U11 pad c11: /TARGET_RX -> /TMS
- U11 pad c12: /TARGET_TX -> /TDO
- U11 pad c13: /EN_PWR_22 -> /TDI
- U11 pad c14: /EN_ICSP_22 -> +5V
- U11 pad c15: /EN_JTAG_22 -> +3V3
- U11 pad c16: /SPARE_22 -> GND
- U11 pad c2: +3V3 -> /EN_JTAG_21
- U11 pad c3: +5V -> /EN_ICSP_21
- U11 pad c4: /TDI -> /EN_PWR_21
- U11 pad c5: /TDO -> /TARGET_TX
- U11 pad c6: /TMS -> /TARGET_RX
- U11 pad c7: /TCK -> /PGED
- U11 pad c8: /~MCLR~ -> /PGEC
- U11 pad c9: /PGEC -> /~MCLR~
- U12 pad a1: GND -> /SPARE_24
- U12 pad a10: /PGED -> /TCK
- U12 pad a11: /TARGET_RX -> /TMS
- U12 pad a12: /TARGET_TX -> /TDO
- U12 pad a13: /EN_PWR_23 -> /TDI
- U12 pad a14: /EN_ICSP_23 -> +5V
- U12 pad a15: /EN_JTAG_23 -> +3V3
- U12 pad a16: /SPARE_23 -> GND
- U12 pad a2: +3V3 -> /EN_JTAG_24
- U12 pad a3: +5V -> /EN_ICSP_24
- U12 pad a4: /TDI -> /EN_PWR_24
- U12 pad a5: /TDO -> /TARGET_TX
- U12 pad a6: /TMS -> /TARGET_RX
- U12 pad a7: /TCK -> /PGED
- U12 pad a8: /~MCLR~ -> /PGEC
- U12 pad a9: /PGEC -> /~MCLR~
- U12 pad b1: GND -> (no net)
- U12 pad b10: /PGED -> /TCK
- U12 pad b11: /TARGET_RX -> /TMS
- U12 pad b12: /TARGET_TX -> /TDO
- U12 pad b13: (no net) -> /TDI
- U12 pad b14: (no net) -> +5V
- U12 pad b15: (no net) -> +3V3
- U12 pad b16: (no net) -> GND
- U12 pad b2: +3V3 -> (no net)
- U12 pad b3: +5V -> (no net)
- U12 pad b4: /TDI -> (no net)
- U12 pad b5: /TDO -> /TARGET_TX
- U12 pad b6: /TMS -> /TARGET_RX
- U12 pad b7: /TCK -> /PGED
- U12 pad b8: /~MCLR~ -> /PGEC
- U12 pad b9: /PGEC -> /~MCLR~
- U12 pad c1: GND -> /SPARE_23
- U12 pad c10: /PGED -> /TCK
- U12 pad c11: /TARGET_RX -> /TMS
- U12 pad c12: /TARGET_TX -> /TDO
- U12 pad c13: /EN_PWR_24 -> /TDI
- U12 pad c14: /EN_ICSP_24 -> +5V
- U12 pad c15: /EN_JTAG_24 -> +3V3
- U12 pad c16: /SPARE_24 -> GND
- U12 pad c2: +3V3 -> /EN_JTAG_23
- U12 pad c3: +5V -> /EN_ICSP_23
- U12 pad c4: /TDI -> /EN_PWR_23
- U12 pad c5: /TDO -> /TARGET_TX
- U12 pad c6: /TMS -> /TARGET_RX
- U12 pad c7: /TCK -> /PGED
- U12 pad c8: /~MCLR~ -> /PGEC
- U12 pad c9: /PGEC -> /~MCLR~
- U13 pad a1: GND -> /SPARE_26
- U13 pad a10: /PGED -> /TCK
- U13 pad a11: /TARGET_RX -> /TMS
- U13 pad a12: /TARGET_TX -> /TDO
- U13 pad a13: /EN_PWR_25 -> /TDI
- U13 pad a14: /EN_ICSP_25 -> +5V
- U13 pad a15: /EN_JTAG_25 -> +3V3
- U13 pad a16: /SPARE_25 -> GND
- U13 pad a2: +3V3 -> /EN_JTAG_26
- U13 pad a3: +5V -> /EN_ICSP_26
- U13 pad a4: /TDI -> /EN_PWR_26
- U13 pad a5: /TDO -> /TARGET_TX
- U13 pad a6: /TMS -> /TARGET_RX
- U13 pad a7: /TCK -> /PGED
- U13 pad a8: /~MCLR~ -> /PGEC
- U13 pad a9: /PGEC -> /~MCLR~
- U13 pad b1: GND -> (no net)
- U13 pad b10: /PGED -> /TCK
- U13 pad b11: /TARGET_RX -> /TMS
- U13 pad b12: /TARGET_TX -> /TDO
- U13 pad b13: (no net) -> /TDI
- U13 pad b14: (no net) -> +5V
- U13 pad b15: (no net) -> +3V3
- U13 pad b16: (no net) -> GND
- U13 pad b2: +3V3 -> (no net)
- U13 pad b3: +5V -> (no net)
- U13 pad b4: /TDI -> (no net)
- U13 pad b5: /TDO -> /TARGET_TX
- U13 pad b6: /TMS -> /TARGET_RX
- U13 pad b7: /TCK -> /PGED
- U13 pad b8: /~MCLR~ -> /PGEC
- U13 pad b9: /PGEC -> /~MCLR~
- U13 pad c1: GND -> /SPARE_25
- U13 pad c10: /PGED -> /TCK
- U13 pad c11: /TARGET_RX -> /TMS
- U13 pad c12: /TARGET_TX -> /TDO
- U13 pad c13: /EN_PWR_26 -> /TDI
- U13 pad c14: /EN_ICSP_26 -> +5V
- U13 pad c15: /EN_JTAG_26 -> +3V3
- U13 pad c16: /SPARE_26 -> GND
- U13 pad c2: +3V3 -> /EN_JTAG_25
- U13 pad c3: +5V -> /EN_ICSP_25
- U13 pad c4: /TDI -> /EN_PWR_25
- U13 pad c5: /TDO -> /TARGET_TX
- U13 pad c6: /TMS -> /TARGET_RX
- U13 pad c7: /TCK -> /PGED
- U13 pad c8: /~MCLR~ -> /PGEC
- U13 pad c9: /PGEC -> /~MCLR~
- U14 pad a1: GND -> /SPARE_28
- U14 pad a10: /PGED -> /TCK
- U14 pad a11: /TARGET_RX -> /TMS
- U14 pad a12: /TARGET_TX -> /TDO
- U14 pad a13: /EN_PWR_27 -> /TDI
- U14 pad a14: /EN_ICSP_27 -> +5V
- U14 pad a15: /EN_JTAG_27 -> +3V3
- U14 pad a16: /SPARE_27 -> GND
- U14 pad a2: +3V3 -> /EN_JTAG_28
- U14 pad a3: +5V -> /EN_ICSP_28
- U14 pad a4: /TDI -> /EN_PWR_28
- U14 pad a5: /TDO -> /TARGET_TX
- U14 pad a6: /TMS -> /TARGET_RX
- U14 pad a7: /TCK -> /PGED
- U14 pad a8: /~MCLR~ -> /PGEC
- U14 pad a9: /PGEC -> /~MCLR~
- U14 pad b1: GND -> (no net)
- U14 pad b10: /PGED -> /TCK
- U14 pad b11: /TARGET_RX -> /TMS
- U14 pad b12: /TARGET_TX -> /TDO
- U14 pad b13: (no net) -> /TDI
- U14 pad b14: (no net) -> +5V
- U14 pad b15: (no net) -> +3V3
- U14 pad b16: (no net) -> GND
- U14 pad b2: +3V3 -> (no net)
- U14 pad b3: +5V -> (no net)
- U14 pad b4: /TDI -> (no net)
- U14 pad b5: /TDO -> /TARGET_TX
- U14 pad b6: /TMS -> /TARGET_RX
- U14 pad b7: /TCK -> /PGED
- U14 pad b8: /~MCLR~ -> /PGEC
- U14 pad b9: /PGEC -> /~MCLR~
- U14 pad c1: GND -> /SPARE_27
- U14 pad c10: /PGED -> /TCK
- U14 pad c11: /TARGET_RX -> /TMS
- U14 pad c12: /TARGET_TX -> /TDO
- U14 pad c13: /EN_PWR_28 -> /TDI
- U14 pad c14: /EN_ICSP_28 -> +5V
- U14 pad c15: /EN_JTAG_28 -> +3V3
- U14 pad c16: /SPARE_28 -> GND
- U14 pad c2: +3V3 -> /EN_JTAG_27
- U14 pad c3: +5V -> /EN_ICSP_27
- U14 pad c4: /TDI -> /EN_PWR_27
- U14 pad c5: /TDO -> /TARGET_TX
- U14 pad c6: /TMS -> /TARGET_RX
- U14 pad c7: /TCK -> /PGED
- U14 pad c8: /~MCLR~ -> /PGEC
- U14 pad c9: /PGEC -> /~MCLR~
- U15 pad a1: GND -> /SPARE_30
- U15 pad a10: /PGED -> /TCK
- U15 pad a11: /TARGET_RX -> /TMS
- U15 pad a12: /TARGET_TX -> /TDO
- U15 pad a13: /EN_PWR_29 -> /TDI
- U15 pad a14: /EN_ICSP_29 -> +5V
- U15 pad a15: /EN_JTAG_29 -> +3V3
- U15 pad a16: /SPARE_29 -> GND
- U15 pad a2: +3V3 -> /EN_JTAG_30
- U15 pad a3: +5V -> /EN_ICSP_30
- U15 pad a4: /TDI -> /EN_PWR_30
- U15 pad a5: /TDO -> /TARGET_TX
- U15 pad a6: /TMS -> /TARGET_RX
- U15 pad a7: /TCK -> /PGED
- U15 pad a8: /~MCLR~ -> /PGEC
- U15 pad a9: /PGEC -> /~MCLR~
- U15 pad b1: GND -> (no net)
- U15 pad b10: /PGED -> /TCK
- U15 pad b11: /TARGET_RX -> /TMS
- U15 pad b12: /TARGET_TX -> /TDO
- U15 pad b13: (no net) -> /TDI
- U15 pad b14: (no net) -> +5V
- U15 pad b15: (no net) -> +3V3
- U15 pad b16: (no net) -> GND
- U15 pad b2: +3V3 -> (no net)
- U15 pad b3: +5V -> (no net)
- U15 pad b4: /TDI -> (no net)
- U15 pad b5: /TDO -> /TARGET_TX
- U15 pad b6: /TMS -> /TARGET_RX
- U15 pad b7: /TCK -> /PGED
- U15 pad b8: /~MCLR~ -> /PGEC
- U15 pad b9: /PGEC -> /~MCLR~
- U15 pad c1: GND -> /SPARE_29
- U15 pad c10: /PGED -> /TCK
- U15 pad c11: /TARGET_RX -> /TMS
- U15 pad c12: /TARGET_TX -> /TDO
- U15 pad c13: /EN_PWR_30 -> /TDI
- U15 pad c14: /EN_ICSP_30 -> +5V
- U15 pad c15: /EN_JTAG_30 -> +3V3
- U15 pad c16: /SPARE_30 -> GND
- U15 pad c2: +3V3 -> /EN_JTAG_29
- U15 pad c3: +5V -> /EN_ICSP_29
- U15 pad c4: /TDI -> /EN_PWR_29
- U15 pad c5: /TDO -> /TARGET_TX
- U15 pad c6: /TMS -> /TARGET_RX
- U15 pad c7: /TCK -> /PGED
- U15 pad c8: /~MCLR~ -> /PGEC
- U15 pad c9: /PGEC -> /~MCLR~
- U16 pad a1: GND -> /SPARE_32
- U16 pad a10: /PGED -> /TCK
- U16 pad a11: /TARGET_RX -> /TMS
- U16 pad a12: /TARGET_TX -> /TDO
- U16 pad a13: /EN_PWR_31 -> /TDI
- U16 pad a14: /EN_ICSP_31 -> +5V
- U16 pad a15: /EN_JTAG_31 -> +3V3
- U16 pad a16: /SPARE_31 -> GND
- U16 pad a2: +3V3 -> /EN_JTAG_32
- U16 pad a3: +5V -> /EN_ICSP_32
- U16 pad a4: /TDI -> /EN_PWR_32
- U16 pad a5: /TDO -> /TARGET_TX
- U16 pad a6: /TMS -> /TARGET_RX
- U16 pad a7: /TCK -> /PGED
- U16 pad a8: /~MCLR~ -> /PGEC
- U16 pad a9: /PGEC -> /~MCLR~
- U16 pad b1: GND -> (no net)
- U16 pad b10: /PGED -> /TCK
- U16 pad b11: /TARGET_RX -> /TMS
- U16 pad b12: /TARGET_TX -> /TDO
- U16 pad b13: (no net) -> /TDI
- U16 pad b14: (no net) -> +5V
- U16 pad b15: (no net) -> +3V3
- U16 pad b16: (no net) -> GND
- U16 pad b2: +3V3 -> (no net)
- U16 pad b3: +5V -> (no net)
- U16 pad b4: /TDI -> (no net)
- U16 pad b5: /TDO -> /TARGET_TX
- U16 pad b6: /TMS -> /TARGET_RX
- U16 pad b7: /TCK -> /PGED
- U16 pad b8: /~MCLR~ -> /PGEC
- U16 pad b9: /PGEC -> /~MCLR~
- U16 pad c1: GND -> /SPARE_31
- U16 pad c10: /PGED -> /TCK
- U16 pad c11: /TARGET_RX -> /TMS
- U16 pad c12: /TARGET_TX -> /TDO
- U16 pad c13: /EN_PWR_32 -> /TDI
- U16 pad c14: /EN_ICSP_32 -> +5V
- U16 pad c15: /EN_JTAG_32 -> +3V3
- U16 pad c16: /SPARE_32 -> GND
- U16 pad c2: +3V3 -> /EN_JTAG_31
- U16 pad c3: +5V -> /EN_ICSP_31
- U16 pad c4: /TDI -> /EN_PWR_31
- U16 pad c5: /TDO -> /TARGET_TX
- U16 pad c6: /TMS -> /TARGET_RX
- U16 pad c7: /TCK -> /PGED
- U16 pad c8: /~MCLR~ -> /PGEC
- U16 pad c9: /PGEC -> /~MCLR~
- U17 pad a1: GND -> /SPARE_34
- U17 pad a10: /PGED -> /TCK
- U17 pad a11: /TARGET_RX -> /TMS
- U17 pad a12: /TARGET_TX -> /TDO
- U17 pad a13: /EN_PWR_33 -> /TDI
- U17 pad a14: /EN_ICSP_33 -> +5V
- U17 pad a15: /EN_JTAG_33 -> +3V3
- U17 pad a16: /SPARE_33 -> GND
- U17 pad a2: +3V3 -> /EN_JTAG_34
- U17 pad a3: +5V -> /EN_ICSP_34
- U17 pad a4: /TDI -> /EN_PWR_34
- U17 pad a5: /TDO -> /TARGET_TX
- U17 pad a6: /TMS -> /TARGET_RX
- U17 pad a7: /TCK -> /PGED
- U17 pad a8: /~MCLR~ -> /PGEC
- U17 pad a9: /PGEC -> /~MCLR~
- U17 pad b1: GND -> (no net)
- U17 pad b10: /PGED -> /TCK
- U17 pad b11: /TARGET_RX -> /TMS
- U17 pad b12: /TARGET_TX -> /TDO
- U17 pad b13: (no net) -> /TDI
- U17 pad b14: (no net) -> +5V
- U17 pad b15: (no net) -> +3V3
- U17 pad b16: (no net) -> GND
- U17 pad b2: +3V3 -> (no net)
- U17 pad b3: +5V -> (no net)
- U17 pad b4: /TDI -> (no net)
- U17 pad b5: /TDO -> /TARGET_TX
- U17 pad b6: /TMS -> /TARGET_RX
- U17 pad b7: /TCK -> /PGED
- U17 pad b8: /~MCLR~ -> /PGEC
- U17 pad b9: /PGEC -> /~MCLR~
- U17 pad c1: GND -> /SPARE_33
- U17 pad c10: /PGED -> /TCK
- U17 pad c11: /TARGET_RX -> /TMS
- U17 pad c12: /TARGET_TX -> /TDO
- U17 pad c13: /EN_PWR_34 -> /TDI
- U17 pad c14: /EN_ICSP_34 -> +5V
- U17 pad c15: /EN_JTAG_34 -> +3V3
- U17 pad c16: /SPARE_34 -> GND
- U17 pad c2: +3V3 -> /EN_JTAG_33
- U17 pad c3: +5V -> /EN_ICSP_33
- U17 pad c4: /TDI -> /EN_PWR_33
- U17 pad c5: /TDO -> /TARGET_TX
- U17 pad c6: /TMS -> /TARGET_RX
- U17 pad c7: /TCK -> /PGED
- U17 pad c8: /~MCLR~ -> /PGEC
- U17 pad c9: /PGEC -> /~MCLR~
- U18 pad a1: GND -> (no net)
- U18 pad a10: /PGED -> /TCK
- U18 pad a11: /TARGET_RX -> /TMS
- U18 pad a12: /TARGET_TX -> /TDO
- U18 pad a13: /DATA_IN_1 -> /TDI
- U18 pad a14: /SHIFT_CLK_IN -> +5V
- U18 pad a15: /STORAGE_CLK -> +3V3
- U18 pad a16: /~OE~ -> GND
- U18 pad a2: +3V3 -> /EN_JTAG_36
- U18 pad a3: +5V -> /EN_ICSP_36
- U18 pad a4: /TDI -> /~MASTER_RST~
- U18 pad a5: /TDO -> /TARGET_TX
- U18 pad a6: /TMS -> /TARGET_RX
- U18 pad a7: /TCK -> /PGED
- U18 pad a8: /~MCLR~ -> /PGEC
- U18 pad a9: /PGEC -> /~MCLR~
- U18 pad b1: GND -> (no net)
- U18 pad b10: /PGED -> /TCK
- U18 pad b11: /TARGET_RX -> /TMS
- U18 pad b12: /TARGET_TX -> /TDO
- U18 pad b13: (no net) -> /TDI
- U18 pad b14: (no net) -> +5V
- U18 pad b15: (no net) -> +3V3
- U18 pad b16: (no net) -> GND
- U18 pad b2: +3V3 -> (no net)
- U18 pad b3: +5V -> (no net)
- U18 pad b4: /TDI -> (no net)
- U18 pad b5: /TDO -> /TARGET_TX
- U18 pad b6: /TMS -> /TARGET_RX
- U18 pad b7: /TCK -> /PGED
- U18 pad b8: /~MCLR~ -> /PGEC
- U18 pad b9: /PGEC -> /~MCLR~
- U18 pad c1: GND -> /~OE~
- U18 pad c10: /PGED -> /TCK
- U18 pad c11: /TARGET_RX -> /TMS
- U18 pad c12: /TARGET_TX -> /TDO
- U18 pad c13: /~MASTER_RST~ -> /TDI
- U18 pad c14: /EN_ICSP_36 -> +5V
- U18 pad c15: /EN_JTAG_36 -> +3V3
- U18 pad c16: (no net) -> GND
- U18 pad c2: +3V3 -> /STORAGE_CLK
- U18 pad c3: +5V -> /SHIFT_CLK_IN
- U18 pad c4: /TDI -> /DATA_IN_1
- U18 pad c5: /TDO -> /TARGET_TX
- U18 pad c6: /TMS -> /TARGET_RX
- U18 pad c7: /TCK -> /PGED
- U18 pad c8: /~MCLR~ -> /PGEC
- U18 pad c9: /PGEC -> /~MCLR~
- U19 pad a1: GND -> (no net)
- U19 pad a10: /PGED -> (no net)
- U19 pad a11: /TARGET_RX -> (no net)
- U19 pad a12: /TARGET_TX -> (no net)
- U19 pad a13: /EN_PWR_37 -> (no net)
- U19 pad a14: /EN_ICSP_37 -> +5V
- U19 pad a15: /EN_JTAG_37 -> +3V3
- U19 pad a16: /SPARE_37 -> GND
- U19 pad a2: +3V3 -> (no net)
- U19 pad a3: +5V -> (no net)
- U19 pad a4: /TDI -> (no net)
- U19 pad a5: /TDO -> (no net)
- U19 pad a6: /TMS -> (no net)
- U19 pad a7: /TCK -> (no net)
- U19 pad a8: /~MCLR~ -> (no net)
- U19 pad a9: /PGEC -> (no net)
- U19 pad b1: GND -> (no net)
- U19 pad b14: (no net) -> +5V
- U19 pad b15: (no net) -> +3V3
- U19 pad b16: (no net) -> GND
- U19 pad b2: +3V3 -> (no net)
- U19 pad b3: +5V -> (no net)
- U19 pad c1: GND -> /SPARE_37
- U19 pad c10: (no net) -> /TCK
- U19 pad c11: (no net) -> /TMS
- U19 pad c12: (no net) -> /TDO
- U19 pad c13: (no net) -> /TDI
- U19 pad c14: (no net) -> +5V
- U19 pad c15: (no net) -> +3V3
- U19 pad c16: (no net) -> GND
- U19 pad c2: +3V3 -> /EN_JTAG_37
- U19 pad c3: +5V -> /EN_ICSP_37
- U19 pad c4: (no net) -> /EN_PWR_37
- U19 pad c5: (no net) -> /TARGET_TX
- U19 pad c6: (no net) -> /TARGET_RX
- U19 pad c7: (no net) -> /PGED
- U19 pad c8: (no net) -> /PGEC
- U19 pad c9: (no net) -> /~MCLR~
- U2 pad a1: GND -> /SPARE_4
- U2 pad a10: /PGED -> /TCK
- U2 pad a11: /TARGET_RX -> /TMS
- U2 pad a12: /TARGET_TX -> /TDO
- U2 pad a13: /EN_PWR_3 -> /TDI
- U2 pad a14: /EN_ICSP_3 -> +5V
- U2 pad a15: /EN_JTAG_3 -> +3V3
- U2 pad a16: /SPARE_3 -> GND
- U2 pad a2: +3V3 -> /EN_JTAG_4
- U2 pad a3: +5V -> /EN_ICSP_4
- U2 pad a4: /TDI -> /EN_PWR_4
- U2 pad a5: /TDO -> /TARGET_TX
- U2 pad a6: /TMS -> /TARGET_RX
- U2 pad a7: /TCK -> /PGED
- U2 pad a8: /~MCLR~ -> /PGEC
- U2 pad a9: /PGEC -> /~MCLR~
- U2 pad b1: GND -> (no net)
- U2 pad b10: /PGED -> /TCK
- U2 pad b11: /TARGET_RX -> /TMS
- U2 pad b12: /TARGET_TX -> /TDO
- U2 pad b13: (no net) -> /TDI
- U2 pad b14: (no net) -> +5V
- U2 pad b15: (no net) -> +3V3
- U2 pad b16: (no net) -> GND
- U2 pad b2: +3V3 -> (no net)
- U2 pad b3: +5V -> (no net)
- U2 pad b4: /TDI -> (no net)
- U2 pad b5: /TDO -> /TARGET_TX
- U2 pad b6: /TMS -> /TARGET_RX
- U2 pad b7: /TCK -> /PGED
- U2 pad b8: /~MCLR~ -> /PGEC
- U2 pad b9: /PGEC -> /~MCLR~
- U2 pad c1: GND -> /SPARE_3
- U2 pad c10: /PGED -> /TCK
- U2 pad c11: /TARGET_RX -> /TMS
- U2 pad c12: /TARGET_TX -> /TDO
- U2 pad c13: /EN_PWR_4 -> /TDI
- U2 pad c14: /EN_ICSP_4 -> +5V
- U2 pad c15: /EN_JTAG_4 -> +3V3
- U2 pad c16: /SPARE_4 -> GND
- U2 pad c2: +3V3 -> /EN_JTAG_3
- U2 pad c3: +5V -> /EN_ICSP_3
- U2 pad c4: /TDI -> /EN_PWR_3
- U2 pad c5: /TDO -> /TARGET_TX
- U2 pad c6: /TMS -> /TARGET_RX
- U2 pad c7: /TCK -> /PGED
- U2 pad c8: /~MCLR~ -> /PGEC
- U2 pad c9: /PGEC -> /~MCLR~
- U20 pad a1: GND -> /~OE~
- U20 pad a10: /PGED -> (no net)
- U20 pad a11: /TARGET_RX -> (no net)
- U20 pad a12: /TARGET_TX -> (no net)
- U20 pad a13: /EN_PWR_39 -> (no net)
- U20 pad a14: /EN_ICSP_39 -> +5V
- U20 pad a15: /EN_JTAG_39 -> +3V3
- U20 pad a16: /SPARE_39 -> GND
- U20 pad a2: +3V3 -> /STORAGE_CLK
- U20 pad a3: +5V -> /SHIFT_CLK_IN
- U20 pad a4: /TDI -> /DATA_IN_1
- U20 pad a5: /TDO -> /~MASTER_RST~
- U20 pad a6: /TMS -> (no net)
- U20 pad a7: /TCK -> (no net)
- U20 pad a8: /~MCLR~ -> (no net)
- U20 pad a9: /PGEC -> (no net)
- U20 pad b1: GND -> (no net)
- U20 pad b14: (no net) -> +5V
- U20 pad b15: (no net) -> +3V3
- U20 pad b16: (no net) -> GND
- U20 pad b2: +3V3 -> (no net)
- U20 pad b3: +5V -> (no net)
- U20 pad c1: GND -> /SPARE_39
- U20 pad c10: (no net) -> /TCK
- U20 pad c11: (no net) -> /TMS
- U20 pad c12: /~MASTER_RST~ -> /TDO
- U20 pad c13: /DATA_IN_1 -> /TDI
- U20 pad c14: /SHIFT_CLK_IN -> +5V
- U20 pad c15: /STORAGE_CLK -> +3V3
- U20 pad c16: /~OE~ -> GND
- U20 pad c2: +3V3 -> /EN_JTAG_39
- U20 pad c3: +5V -> /EN_ICSP_39
- U20 pad c4: (no net) -> /EN_PWR_39
- U20 pad c5: (no net) -> /TARGET_TX
- U20 pad c6: (no net) -> /TARGET_RX
- U20 pad c7: (no net) -> /PGED
- U20 pad c8: (no net) -> /PGEC
- U20 pad c9: (no net) -> /~MCLR~
- U3 pad a1: GND -> /SPARE_6
- U3 pad a10: /PGED -> /TCK
- U3 pad a11: /TARGET_RX -> /TMS
- U3 pad a12: /TARGET_TX -> /TDO
- U3 pad a13: /EN_PWR_5 -> /TDI
- U3 pad a14: /EN_ICSP_5 -> +5V
- U3 pad a15: /EN_JTAG_5 -> +3V3
- U3 pad a16: /SPARE_5 -> GND
- U3 pad a2: +3V3 -> /EN_JTAG_6
- U3 pad a3: +5V -> /EN_ICSP_6
- U3 pad a4: /TDI -> /EN_PWR_6
- U3 pad a5: /TDO -> /TARGET_TX
- U3 pad a6: /TMS -> /TARGET_RX
- U3 pad a7: /TCK -> /PGED
- U3 pad a8: /~MCLR~ -> /PGEC
- U3 pad a9: /PGEC -> /~MCLR~
- U3 pad b1: GND -> (no net)
- U3 pad b10: /PGED -> /TCK
- U3 pad b11: /TARGET_RX -> /TMS
- U3 pad b12: /TARGET_TX -> /TDO
- U3 pad b13: (no net) -> /TDI
- U3 pad b14: (no net) -> +5V
- U3 pad b15: (no net) -> +3V3
- U3 pad b16: (no net) -> GND
- U3 pad b2: +3V3 -> (no net)
- U3 pad b3: +5V -> (no net)
- U3 pad b4: /TDI -> (no net)
- U3 pad b5: /TDO -> /TARGET_TX
- U3 pad b6: /TMS -> /TARGET_RX
- U3 pad b7: /TCK -> /PGED
- U3 pad b8: /~MCLR~ -> /PGEC
- U3 pad b9: /PGEC -> /~MCLR~
- U3 pad c1: GND -> /SPARE_5
- U3 pad c10: /PGED -> /TCK
- U3 pad c11: /TARGET_RX -> /TMS
- U3 pad c12: /TARGET_TX -> /TDO
- U3 pad c13: /EN_PWR_6 -> /TDI
- U3 pad c14: /EN_ICSP_6 -> +5V
- U3 pad c15: /EN_JTAG_6 -> +3V3
- U3 pad c16: /SPARE_6 -> GND
- U3 pad c2: +3V3 -> /EN_JTAG_5
- U3 pad c3: +5V -> /EN_ICSP_5
- U3 pad c4: /TDI -> /EN_PWR_5
- U3 pad c5: /TDO -> /TARGET_TX
- U3 pad c6: /TMS -> /TARGET_RX
- U3 pad c7: /TCK -> /PGED
- U3 pad c8: /~MCLR~ -> /PGEC
- U3 pad c9: /PGEC -> /~MCLR~
- U4 pad a1: GND -> /SPARE_8
- U4 pad a10: /PGED -> /TCK
- U4 pad a11: /TARGET_RX -> /TMS
- U4 pad a12: /TARGET_TX -> /TDO
- U4 pad a13: /EN_PWR_7 -> /TDI
- U4 pad a14: /EN_ICSP_7 -> +5V
- U4 pad a15: /EN_JTAG_7 -> +3V3
- U4 pad a16: /SPARE_7 -> GND
- U4 pad a2: +3V3 -> /EN_JTAG_8
- U4 pad a3: +5V -> /EN_ICSP_8
- U4 pad a4: /TDI -> /EN_PWR_8
- U4 pad a5: /TDO -> /TARGET_TX
- U4 pad a6: /TMS -> /TARGET_RX
- U4 pad a7: /TCK -> /PGED
- U4 pad a8: /~MCLR~ -> /PGEC
- U4 pad a9: /PGEC -> /~MCLR~
- U4 pad b1: GND -> (no net)
- U4 pad b10: /PGED -> /TCK
- U4 pad b11: /TARGET_RX -> /TMS
- U4 pad b12: /TARGET_TX -> /TDO
- U4 pad b13: (no net) -> /TDI
- U4 pad b14: (no net) -> +5V
- U4 pad b15: (no net) -> +3V3
- U4 pad b16: (no net) -> GND
- U4 pad b2: +3V3 -> (no net)
- U4 pad b3: +5V -> (no net)
- U4 pad b4: /TDI -> (no net)
- U4 pad b5: /TDO -> /TARGET_TX
- U4 pad b6: /TMS -> /TARGET_RX
- U4 pad b7: /TCK -> /PGED
- U4 pad b8: /~MCLR~ -> /PGEC
- U4 pad b9: /PGEC -> /~MCLR~
- U4 pad c1: GND -> /SPARE_7
- U4 pad c10: /PGED -> /TCK
- U4 pad c11: /TARGET_RX -> /TMS
- U4 pad c12: /TARGET_TX -> /TDO
- U4 pad c13: /EN_PWR_8 -> /TDI
- U4 pad c14: /EN_ICSP_8 -> +5V
- U4 pad c15: /EN_JTAG_8 -> +3V3
- U4 pad c16: /SPARE_8 -> GND
- U4 pad c2: +3V3 -> /EN_JTAG_7
- U4 pad c3: +5V -> /EN_ICSP_7
- U4 pad c4: /TDI -> /EN_PWR_7
- U4 pad c5: /TDO -> /TARGET_TX
- U4 pad c6: /TMS -> /TARGET_RX
- U4 pad c7: /TCK -> /PGED
- U4 pad c8: /~MCLR~ -> /PGEC
- U4 pad c9: /PGEC -> /~MCLR~
- U5 pad a1: GND -> /SPARE_10
- U5 pad a10: /PGED -> /TCK
- U5 pad a11: /TARGET_RX -> /TMS
- U5 pad a12: /TARGET_TX -> /TDO
- U5 pad a13: /EN_PWR_9 -> /TDI
- U5 pad a14: /EN_ICSP_9 -> +5V
- U5 pad a15: /EN_JTAG_9 -> +3V3
- U5 pad a16: /SPARE_9 -> GND
- U5 pad a2: +3V3 -> /EN_JTAG_10
- U5 pad a3: +5V -> /EN_ICSP_10
- U5 pad a4: /TDI -> /EN_PWR_10
- U5 pad a5: /TDO -> /TARGET_TX
- U5 pad a6: /TMS -> /TARGET_RX
- U5 pad a7: /TCK -> /PGED
- U5 pad a8: /~MCLR~ -> /PGEC
- U5 pad a9: /PGEC -> /~MCLR~
- U5 pad b1: GND -> (no net)
- U5 pad b10: /PGED -> /TCK
- U5 pad b11: /TARGET_RX -> /TMS
- U5 pad b12: /TARGET_TX -> /TDO
- U5 pad b13: (no net) -> /TDI
- U5 pad b14: (no net) -> +5V
- U5 pad b15: (no net) -> +3V3
- U5 pad b16: (no net) -> GND
- U5 pad b2: +3V3 -> (no net)
- U5 pad b3: +5V -> (no net)
- U5 pad b4: /TDI -> (no net)
- U5 pad b5: /TDO -> /TARGET_TX
- U5 pad b6: /TMS -> /TARGET_RX
- U5 pad b7: /TCK -> /PGED
- U5 pad b8: /~MCLR~ -> /PGEC
- U5 pad b9: /PGEC -> /~MCLR~
- U5 pad c1: GND -> /SPARE_9
- U5 pad c10: /PGED -> /TCK
- U5 pad c11: /TARGET_RX -> /TMS
- U5 pad c12: /TARGET_TX -> /TDO
- U5 pad c13: /EN_PWR_10 -> /TDI
- U5 pad c14: /EN_ICSP_10 -> +5V
- U5 pad c15: /EN_JTAG_10 -> +3V3
- U5 pad c16: /SPARE_10 -> GND
- U5 pad c2: +3V3 -> /EN_JTAG_9
- U5 pad c3: +5V -> /EN_ICSP_9
- U5 pad c4: /TDI -> /EN_PWR_9
- U5 pad c5: /TDO -> /TARGET_TX
- U5 pad c6: /TMS -> /TARGET_RX
- U5 pad c7: /TCK -> /PGED
- U5 pad c8: /~MCLR~ -> /PGEC
- U5 pad c9: /PGEC -> /~MCLR~
- U6 pad a1: GND -> /SPARE_12
- U6 pad a10: /PGED -> /TCK
- U6 pad a11: /TARGET_RX -> /TMS
- U6 pad a12: /TARGET_TX -> /TDO
- U6 pad a13: /EN_PWR_11 -> /TDI
- U6 pad a14: /EN_ICSP_11 -> +5V
- U6 pad a15: /EN_JTAG_11 -> +3V3
- U6 pad a16: /SPARE_11 -> GND
- U6 pad a2: +3V3 -> /EN_JTAG_12
- U6 pad a3: +5V -> /EN_ICSP_12
- U6 pad a4: /TDI -> /EN_PWR_12
- U6 pad a5: /TDO -> /TARGET_TX
- U6 pad a6: /TMS -> /TARGET_RX
- U6 pad a7: /TCK -> /PGED
- U6 pad a8: /~MCLR~ -> /PGEC
- U6 pad a9: /PGEC -> /~MCLR~
- U6 pad b1: GND -> (no net)
- U6 pad b10: /PGED -> /TCK
- U6 pad b11: /TARGET_RX -> /TMS
- U6 pad b12: /TARGET_TX -> /TDO
- U6 pad b13: (no net) -> /TDI
- U6 pad b14: (no net) -> +5V
- U6 pad b15: (no net) -> +3V3
- U6 pad b16: (no net) -> GND
- U6 pad b2: +3V3 -> (no net)
- U6 pad b3: +5V -> (no net)
- U6 pad b4: /TDI -> (no net)
- U6 pad b5: /TDO -> /TARGET_TX
- U6 pad b6: /TMS -> /TARGET_RX
- U6 pad b7: /TCK -> /PGED
- U6 pad b8: /~MCLR~ -> /PGEC
- U6 pad b9: /PGEC -> /~MCLR~
- U6 pad c1: GND -> /SPARE_11
- U6 pad c10: /PGED -> /TCK
- U6 pad c11: /TARGET_RX -> /TMS
- U6 pad c12: /TARGET_TX -> /TDO
- U6 pad c13: /EN_PWR_12 -> /TDI
- U6 pad c14: /EN_ICSP_12 -> +5V
- U6 pad c15: /EN_JTAG_12 -> +3V3
- U6 pad c16: /SPARE_12 -> GND
- U6 pad c2: +3V3 -> /EN_JTAG_11
- U6 pad c3: +5V -> /EN_ICSP_11
- U6 pad c4: /TDI -> /EN_PWR_11
- U6 pad c5: /TDO -> /TARGET_TX
- U6 pad c6: /TMS -> /TARGET_RX
- U6 pad c7: /TCK -> /PGED
- U6 pad c8: /~MCLR~ -> /PGEC
- U6 pad c9: /PGEC -> /~MCLR~
- U7 pad a1: GND -> /SPARE_14
- U7 pad a10: /PGED -> /TCK
- U7 pad a11: /TARGET_RX -> /TMS
- U7 pad a12: /TARGET_TX -> /TDO
- U7 pad a13: /EN_PWR_13 -> /TDI
- U7 pad a14: /EN_ICSP_13 -> +5V
- U7 pad a15: /EN_JTAG_13 -> +3V3
- U7 pad a16: /SPARE_13 -> GND
- U7 pad a2: +3V3 -> /EN_JTAG_14
- U7 pad a3: +5V -> /EN_ICSP_14
- U7 pad a4: /TDI -> /EN_PWR_14
- U7 pad a5: /TDO -> /TARGET_TX
- U7 pad a6: /TMS -> /TARGET_RX
- U7 pad a7: /TCK -> /PGED
- U7 pad a8: /~MCLR~ -> /PGEC
- U7 pad a9: /PGEC -> /~MCLR~
- U7 pad b1: GND -> (no net)
- U7 pad b10: /PGED -> /TCK
- U7 pad b11: /TARGET_RX -> /TMS
- U7 pad b12: /TARGET_TX -> /TDO
- U7 pad b13: (no net) -> /TDI
- U7 pad b14: (no net) -> +5V
- U7 pad b15: (no net) -> +3V3
- U7 pad b16: (no net) -> GND
- U7 pad b2: +3V3 -> (no net)
- U7 pad b3: +5V -> (no net)
- U7 pad b4: /TDI -> (no net)
- U7 pad b5: /TDO -> /TARGET_TX
- U7 pad b6: /TMS -> /TARGET_RX
- U7 pad b7: /TCK -> /PGED
- U7 pad b8: /~MCLR~ -> /PGEC
- U7 pad b9: /PGEC -> /~MCLR~
- U7 pad c1: GND -> /SPARE_13
- U7 pad c10: /PGED -> /TCK
- U7 pad c11: /TARGET_RX -> /TMS
- U7 pad c12: /TARGET_TX -> /TDO
- U7 pad c13: /EN_PWR_14 -> /TDI
- U7 pad c14: /EN_ICSP_14 -> +5V
- U7 pad c15: /EN_JTAG_14 -> +3V3
- U7 pad c16: /SPARE_14 -> GND
- U7 pad c2: +3V3 -> /EN_JTAG_13
- U7 pad c3: +5V -> /EN_ICSP_13
- U7 pad c4: /TDI -> /EN_PWR_13
- U7 pad c5: /TDO -> /TARGET_TX
- U7 pad c6: /TMS -> /TARGET_RX
- U7 pad c7: /TCK -> /PGED
- U7 pad c8: /~MCLR~ -> /PGEC
- U7 pad c9: /PGEC -> /~MCLR~
- U8 pad a1: GND -> /SPARE_16
- U8 pad a10: /PGED -> /TCK
- U8 pad a11: /TARGET_RX -> /TMS
- U8 pad a12: /TARGET_TX -> /TDO
- U8 pad a13: /EN_PWR_15 -> /TDI
- U8 pad a14: /EN_ICSP_15 -> +5V
- U8 pad a15: /EN_JTAG_15 -> +3V3
- U8 pad a16: /SPARE_15 -> GND
- U8 pad a2: +3V3 -> /EN_JTAG_16
- U8 pad a3: +5V -> /EN_ICSP_16
- U8 pad a4: /TDI -> /EN_PWR_16
- U8 pad a5: /TDO -> /TARGET_TX
- U8 pad a6: /TMS -> /TARGET_RX
- U8 pad a7: /TCK -> /PGED
- U8 pad a8: /~MCLR~ -> /PGEC
- U8 pad a9: /PGEC -> /~MCLR~
- U8 pad b1: GND -> (no net)
- U8 pad b10: /PGED -> /TCK
- U8 pad b11: /TARGET_RX -> /TMS
- U8 pad b12: /TARGET_TX -> /TDO
- U8 pad b13: (no net) -> /TDI
- U8 pad b14: (no net) -> +5V
- U8 pad b15: (no net) -> +3V3
- U8 pad b16: (no net) -> GND
- U8 pad b2: +3V3 -> (no net)
- U8 pad b3: +5V -> (no net)
- U8 pad b4: /TDI -> (no net)
- U8 pad b5: /TDO -> /TARGET_TX
- U8 pad b6: /TMS -> /TARGET_RX
- U8 pad b7: /TCK -> /PGED
- U8 pad b8: /~MCLR~ -> /PGEC
- U8 pad b9: /PGEC -> /~MCLR~
- U8 pad c1: GND -> /SPARE_15
- U8 pad c10: /PGED -> /TCK
- U8 pad c11: /TARGET_RX -> /TMS
- U8 pad c12: /TARGET_TX -> /TDO
- U8 pad c13: /EN_PWR_16 -> /TDI
- U8 pad c14: /EN_ICSP_16 -> +5V
- U8 pad c15: /EN_JTAG_16 -> +3V3
- U8 pad c16: /SPARE_16 -> GND
- U8 pad c2: +3V3 -> /EN_JTAG_15
- U8 pad c3: +5V -> /EN_ICSP_15
- U8 pad c4: /TDI -> /EN_PWR_15
- U8 pad c5: /TDO -> /TARGET_TX
- U8 pad c6: /TMS -> /TARGET_RX
- U8 pad c7: /TCK -> /PGED
- U8 pad c8: /~MCLR~ -> /PGEC
- U8 pad c9: /PGEC -> /~MCLR~
- U9 pad a1: GND -> /SPARE_18
- U9 pad a10: /PGED -> /TCK
- U9 pad a11: /TARGET_RX -> /TMS
- U9 pad a12: /TARGET_TX -> /TDO
- U9 pad a13: /EN_PWR_17 -> /TDI
- U9 pad a14: /EN_ICSP_17 -> +5V
- U9 pad a15: /EN_JTAG_17 -> +3V3
- U9 pad a16: /SPARE_17 -> GND
- U9 pad a2: +3V3 -> /EN_JTAG_18
- U9 pad a3: +5V -> /EN_ICSP_18
- U9 pad a4: /TDI -> /EN_PWR_18
- U9 pad a5: /TDO -> /TARGET_TX
- U9 pad a6: /TMS -> /TARGET_RX
- U9 pad a7: /TCK -> /PGED
- U9 pad a8: /~MCLR~ -> /PGEC
- U9 pad a9: /PGEC -> /~MCLR~
- U9 pad b1: GND -> (no net)
- U9 pad b10: /PGED -> /TCK
- U9 pad b11: /TARGET_RX -> /TMS
- U9 pad b12: /TARGET_TX -> /TDO
- U9 pad b13: (no net) -> /TDI
- U9 pad b14: (no net) -> +5V
- U9 pad b15: (no net) -> +3V3
- U9 pad b16: (no net) -> GND
- U9 pad b2: +3V3 -> (no net)
- U9 pad b3: +5V -> (no net)
- U9 pad b4: /TDI -> (no net)
- U9 pad b5: /TDO -> /TARGET_TX
- U9 pad b6: /TMS -> /TARGET_RX
- U9 pad b7: /TCK -> /PGED
- U9 pad b8: /~MCLR~ -> /PGEC
- U9 pad b9: /PGEC -> /~MCLR~
- U9 pad c1: GND -> /SPARE_17
- U9 pad c10: /PGED -> /TCK
- U9 pad c11: /TARGET_RX -> /TMS
- U9 pad c12: /TARGET_TX -> /TDO
- U9 pad c13: /EN_PWR_18 -> /TDI
- U9 pad c14: /EN_ICSP_18 -> +5V
- U9 pad c15: /EN_JTAG_18 -> +3V3
- U9 pad c16: /SPARE_18 -> GND
- U9 pad c2: +3V3 -> /EN_JTAG_17
- U9 pad c3: +5V -> /EN_ICSP_17
- U9 pad c4: /TDI -> /EN_PWR_17
- U9 pad c5: /TDO -> /TARGET_TX
- U9 pad c6: /TMS -> /TARGET_RX
- U9 pad c7: /TCK -> /PGED
- U9 pad c8: /~MCLR~ -> /PGEC
- U9 pad c9: /PGEC -> /~MCLR~
Routing:
- net /EN_PWR_16: track 20.6 -> 24.5 mm
- net /EN_PWR_4: track 20.3 -> 24.3 mm
- net /EN_PWR_8: track 20.5 -> 24.3 mm
- net /EN_PWR_34: track 20.5 -> 24.3 mm
- net /EN_PWR_6: track 20.4 -> 24.2 mm
- net /EN_PWR_2: track 20.8 -> 24.5 mm
- net /EN_PWR_14: track 20.6 -> 24.3 mm
- net /EN_PWR_32: track 20.5 -> 24.2 mm
- net /EN_PWR_10: track 20.3 -> 24.0 mm
- net /EN_PWR_24: track 20.5 -> 24.2 mm
- net /EN_PWR_30: track 20.5 -> 24.1 mm
- net /EN_PWR_26: track 20.5 -> 24.1 mm
- net /EN_PWR_20: track 20.6 -> 24.2 mm
- net /EN_PWR_28: track 20.5 -> 24.1 mm
- net /EN_PWR_22: track 20.5 -> 24.0 mm
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
Commit message: Mid-work commit. Added notes, figured out what works, etc.
Parts:
- H5: moved to B.Cu

Commit message: Update to latest state on primary computer
Connections:
- net /~MASTER_RST~ renamed /~{MASTER_RST}
- net /~MCLR~ renamed /~{MCLR}
- net /~OE~ renamed /~{OE}
Other:
- net class Default removed
