File: RiserCard/RiserCard.sch (KiCad schematic (older format))
At the start: 45 parts, among them J1 Conn_02x05_Odd_Even, J2 Conn_02x05_Odd_Even, J3 Conn_02x05_Odd_Even, J4 Conn_02x05_Odd_Even, J5 Conn_01x01, J6 Conn_01x01, J7 Conn_01x12, J8 Conn_01x12, U1 86094327313755ELF, U2 SN74CBTLV3245ADWR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

Commit message: Mid-work commit. IT's not pretty but it'll work
Connections:
- net +3V3: no longer J7.1 (Pin_1), J8.1 (Pin_1)
- net VCC: now also J7.1 (Pin_1)
- net VDD: now also J8.1 (Pin_1)
Changed lines of the file:
@@
 Wire Wire Line
 	6000 3600 6000 3650
-$Comp
-L power:+3V3 #PWR0152
-U 1 1 61E92B2F
-P 6000 2400
-F 0 "#PWR0152" H 6000 2250 50  0001 C CNN
-F 1 "+3V3" H 6015 2573 50  0000 C CNN
-F 2 "" H 6000 2400 50  0001 C CNN
-F 3 "" H 6000 2400 50  0001 C CNN
-	1    6000 2400
-	1    0    0    -1
-$EndComp
 Wire Wire Line
 	6100 2500 6000 2500
@@
 Wire Wire Line
 	8550 3600 8650 3600
-$Comp
-L power:+3V3 #PWR0154
-U 1 1 62042780
-P 8550 2450
-F 0 "#PWR0154" H 8550 2300 50  0001 C CNN
-F 1 "+3V3" H 8565 2623 50  0000 C CNN
-F 2 "" H 8550 2450 50  0001 C CNN
-F 3 "" H 8550 2450 50  0001 C CNN
-	1    8550 2450
-	1    0    0    -1
-$EndComp
 Wire Wire Line
 	8650 2500 8550 2500
@@
 Text Label 8400 2700 0    50   ~ 0
 B_PGED
+$Comp
+L power:VDD #PWR0152
+U 1 1 620E266B
+P 8550 2450
+F 0 "#PWR0152" H 8550 2300 50  0001 C CNN
+F 1 "VDD" H 8565 2623 50  0000 C CNN
+F 2 "" H 8550 2450 50  0001 C CNN
+F 3 "" H 8550 2450 50  0001 C CNN
+	1    8550 2450
+	1    0    0    -1
+$EndComp
+$Comp
+L power:VCC #PWR0154
+U 1 1 620E7664
+P 6000 2400
+F 0 "#PWR0154" H 6000 2250 50  0001 C CNN
+F 1 "VCC" H 6015 2573 50  0000 C CNN
+F 2 "" H 6000 2400 50  0001 C CNN
+F 3 "" H 6000 2400 50  0001 C CNN
+	1    6000 2400
+	1    0    0    -1
+$EndComp
 $EndSCHEMATC
